File: core.kicad_sch (KiCad schematic)
At the start: 33 parts, among them J11 sync in, Q3 MMBFJ111, U3 OP275, U4 PMP4201Y, U5 CA3140, U6 LM311

Commit message: Revision 2
Parts:
- RV4, RV5: footprint Potentiometer_THT:Potentiometer_Bourns_3296W_Vertical -> Potentiometer_THT:Potentiometer_Bourns_3006P_Horizontal
- renumbered U3 to U5, U4 to U6
