File: input.kicad_sch (KiCad schematic)
At the start: 33 parts, among them J3 CV in, J4 CV in, J5 CV in, SW2 SW_Rotary10, U3 OP275, U8 OPA1679

Commit message: Revision 2
Parts:
- RV3: footprint Potentiometer_THT:Potentiometer_Bourns_3296W_Vertical -> Potentiometer_THT:Potentiometer_Bourns_3006P_Horizontal
- renumbered U8 to U4, U3 to U5
