File: power.kicad_sch (KiCad schematic)
At the start: 32 parts, among them J1 Power input, J2 Daisy chain power, Q1 SQ2348ES, Q2 Si2393DS, U1 LM4040DBZ-10, U11 LM4040DBZ-10, U2 TL072, U3 OP275, U7 TL072, U8 OPA1679

Commit message: Revision 2
Parts:
- removed U2: TL072, Package_SO:SOIC-14_3.9x8.7mm_P1.27mm, symbol Amplifier_Operational:OPA1679
- removed U7: TL072, Package_SO:SOIC-14_3.9x8.7mm_P1.27mm, symbol Amplifier_Operational:TL074
- added C4, C5: 0.1u, Capacitor_SMD:C_0805_2012Metric_Pad1.18x1.45mm_HandSolder, symbol Device:C
- added U10: TL072, Package_SO:SOIC-8_3.9x4.9mm_P1.27mm, symbol Amplifier_Operational:TL072
- added U3: OPA1678, Package_SO:SOIC-8_3.9x4.9mm_P1.27mm, symbol Amplifier_Operational:OPA1678
- added U9: OPA1679, Package_SO:SOIC-14_3.9x8.7mm_P1.27mm, symbol Amplifier_Operational:OPA1679
- renumbered U11 to U2, U3 to U5
Connections:
- net +10V: now also U3.6 (-), U3.7
- net +12V: now also C4.1, U10.8 (V+), U3.8 (V+), U9.4 (V+)
- net -10V: now also U3.1, U3.2 (-)
- net -12V: now also C5.2, U10.4 (V-), U3.4 (V-), U9.11 (V-)
- net GND: now also C4.2, C5.1
- net at C16.1, C30.2, R43.1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: now also U3.3 (+)
- net at C27.2, C3.1, R1.2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: now also U3.5 (+)
Other:
- moved on the sheet: C10, C12, C21, C24, C25, C6, C7, C9, U5C, U8E
