File: vco_1.kicad_pcb (KiCad board)
At the start: 4 copper layers, 80.9 x 99.7 mm, 141 parts, among them J1 Power input, J10 freq out, J11 sync in, J2 Daisy chain power, J3 CV in, J4 CV in, J5 CV in, J6 saw out, J7 tri out, J8 Pulse width input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

Commit message: Revision 2
Parts:
- removed R6: 2k, Resistor_THT:R_Axial_DIN0207_L6.3mm_D2.5mm_P7.62mm_Horizontal
- removed the U2 at (120.7, 89.7)
- removed the U7 at (145.9, 70.1)
- added C4: 0.1u, Capacitor_SMD:C_0805_2012Metric_Pad1.18x1.45mm_HandSolder, F.Cu at (58.9, 80.0)
- added C5: 0.1u, Capacitor_SMD:C_0805_2012Metric_Pad1.18x1.45mm_HandSolder, F.Cu at (44.3, 83.8)
- added TH1: 2k 3300ppm PTC temco, Resistor_THT:R_Axial_DIN0207_L6.3mm_D2.5mm_P7.62mm_Horizontal, F.Cu at (71.1, 122.3)
- added U10: TL072, Package_SO:SOIC-8_3.9x4.9mm_P1.27mm, F.Cu at (51.5, 81.9)
- added U3: OPA1678, Package_SO:SOIC-8_3.9x4.9mm_P1.27mm, F.Cu at (44.8, 118.0)
- added U9: OPA1679, Package_SO:SOIC-14_3.9x8.7mm_P1.27mm, F.Cu at (72.2, 69.2)
- RV3, RV4, RV5, RV6, RV7, RV8, RV9: footprint Potentiometer_THT:Potentiometer_Bourns_3296W_Vertical -> Potentiometer_THT:Potentiometer_Bourns_3006P_Horizontal; moved to B.Cu
- moved J10 105.4 mm to (37.5, 101.6)
- moved U2 104.3 mm to (37.2, 126.2), turned to 180 degrees
- moved R43 95.3 mm to (41.9, 125.0), turned to 0 degrees
- moved C16 95.3 mm to (41.9, 128.5), turned to 0 degrees
- moved C3 94.9 mm to (37.8, 107.8), turned to 180 degrees
- moved C30 90.2 mm to (51.2, 128.8), turned to 0 degrees
- moved TP4 89.0 mm to (51.2, 120.5)
- moved J7 87.6 mm to (47.0, 46.9)
- moved C7 87.0 mm to (46.7, 124.8)
- moved RV4 85.5 mm to (58.8, 118.1), turned to 180 degrees
- moved TP13 84.5 mm to (37.5, 95.9)
- moved J9 84.5 mm to (37.5, 90.2)
- moved TP5 84.0 mm to (37.8, 115.4)
- moved R51 83.8 mm to (37.5, 65.4), turned to 180 degrees
- moved R27 83.6 mm to (50.5, 138.2), turned to 0 degrees
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- renumbered U11 to U2, U8 to U4, U3 to U5, U4 to U6, U5 to U7, U6 to U8
Connections:
- C8 pad 1: Net-(U3A-+) -> Net-(U5A--)
- R20 pad 2: Net-(U3A-+) -> Net-(U5A--)
- R23 pad 2: Net-(U3A-+) -> Net-(U5A--)
- R24 pad 2: Net-(U3A-+) -> Net-(U5A--)
- R25 pad 2: Net-(U3A-+) -> Net-(U5A--)
- R28 pad 2: Net-(U3A-+) -> Net-(U5A--)
- R7 pad 2: Net-(U3A-+) -> Net-(U5A--)
- U5 pad 2: GND -> Net-(U5A--)
- U5 pad 3: Net-(U3A-+) -> GND
Routing:
- net -12V: track 358.1 -> 434.7 mm
- net Net-(U5A--): track 0.00 -> 49.1 mm
- net Net-(U3A-+): track 48.4 -> 0.00 mm
- net +12V: track 356.7 -> 389.0 mm
- net Net-(J9-Pin_1): track 17.8 -> 44.2 mm, vias 0 -> 2
- net Net-(J7-Pin_1): track 18.3 -> 42.9 mm
- net +10V: track 224.5 -> 202.2 mm, vias 12 -> 9
- net -10V: track 152.8 -> 174.0 mm, vias 5 -> 6
- net Net-(U10A-+): track 27.7 -> 9.31 mm, vias 3 -> 0
- net Net-(C11-Pad2): track 15.7 -> 29.5 mm
- net Net-(R37-Pad1): track 6.73 -> 18.3 mm, vias 0 -> 1
- net Net-(J8-Pin_1): track 9.24 -> 20.2 mm
- net Net-(D2-A): track 35.1 -> 44.7 mm
- net /Core/summed_input: track 23.4 -> 31.9 mm
- net Net-(R54-Pad1): track 12.4 -> 4.66 mm
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Other:
- board text added: "VCO 1 Rev 2 Knut Erik Helgesen"
