File: waveshaper.kicad_sch (KiCad schematic)
At the start: 44 parts, among them J10 freq out, J6 saw out, J7 tri out, J8 Pulse width input, J9 pulse out, U10 TL072, U7 TL072

Commit message: Revision 2
Parts:
- removed U10: TL072, Package_SO:SOIC-14_3.9x8.7mm_P1.27mm, symbol Amplifier_Operational:OPA1679
- removed U7: TL072, Package_SO:SOIC-14_3.9x8.7mm_P1.27mm, symbol Amplifier_Operational:TL074
- added U10: TL072, Package_SO:SOIC-8_3.9x4.9mm_P1.27mm, symbol Amplifier_Operational:TL072
- added U9: OPA1679, Package_SO:SOIC-14_3.9x8.7mm_P1.27mm, symbol Amplifier_Operational:OPA1679
- RV6, RV7, RV8, RV9: footprint Potentiometer_THT:Potentiometer_Bourns_3296W_Vertical -> Potentiometer_THT:Potentiometer_Bourns_3006P_Horizontal
Connections:
- net GND: now also U10.5 (+), U9.12 (+), U9.5 (+)
- net at C23.2, RV8.2: now also U9.3 (+)
- net at D2.2 (A), R38.1, RV7.2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: now also U9.8
- net at R38.2, R39.1: now also U9.13 (-)
- net at D3.2 (A), J6.1 (Pin_1), R36.2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: now also U10.2 (-), U10.6 (-)
- net at R54.1: now also U9.7
- net at R46.2, R47.1: now also U9.2 (-)
- net at R53.2, R55.1: now also U9.6 (-)
- net at R52.2, R61.1: now also U10.3 (+)
- net at R36.1: now also U9.14
- net at R49.1: now also U9.1
- net at R53.1: now also U10.1
- net at D4.2 (A): now also U10.7
- net at R34.2, R35.1: now also U9.9 (-)
- net at R33.2: now also U9.10 (+)
